Commit message: Modify some dimentions

File: my_robot/urdf/lidar.xacro (robot description, xacro)
@@ -11,5 +11,5 @@
             <origin xyz="0.0 0.0 0.0" rpy="0.0 0.0 0.0"/>
             <geometry>
-                <box size="0.1 0.1 0.1"/>
+                <mesh filename="package://my_robot/meshes/hokuyo.dae"/>
             </geometry>
         </visual>
@@ -23,5 +23,5 @@
         <parent link="chassis"/>
         <child link="hokuyo"/>
-        <origin xyz="0.15 0.0 0.1" rpy="0.0 0.0 0.0"/>
+        <origin xyz="0.05 0.0 0.1" rpy="0.0 0.0 0.0"/>
     </joint>
 </robot>

File: my_robot/urdf/my_robot.xacro (robot description, xacro)
@@ -27,5 +27,5 @@
       <origin xyz="0 0 0" rpy=" 0 0 0"/>
       <geometry>
-        <box size=".4 .2 .1"/>
+        <box size=".4 .3 .1"/>
       </geometry>
     </visual>
@@ -33,5 +33,5 @@
       <origin xyz="-0.15 0 -0.05" rpy=" 0 0 0"/>
       <geometry>
-        <sphere radius="0.0499"/>
+        <sphere radius="0.05"/>
       </geometry>
     </collision>
@@ -45,5 +45,5 @@
       <origin xyz="0.15 0 -0.05" rpy=" 0 0 0"/>
       <geometry>
-        <sphere radius="0.0499"/>
+        <sphere radius="0.05"/>
       </geometry>
     </collision>
@@ -61,5 +61,5 @@
   <xacro:wheel side="right"/>
   <joint type="continuous" name="left_wheel_hinge">
-            <origin xyz="0 0.15 0" rpy="0 0 0"/>
+            <origin xyz="0 0.19 -0.02" rpy="0 0 0"/>
             <child link="left_wheel"/>
             <parent link="chassis"/>
@@ -69,5 +69,5 @@
           </joint>
   <joint type="continuous" name="right_wheel_hinge">
-            <origin xyz="0 -0.15 0" rpy="0 0 0"/>
+            <origin xyz="0 -0.19 -0.02" rpy="0 0 0"/>
             <child link="right_wheel"/>
             <parent link="chassis"/>

File: my_robot/urdf/wheel.xacro (robot description, xacro)
@@ -6,5 +6,5 @@
                 <origin xyz="0.0 0.0 0.0" rpy="0.0 1.507 1.507"/>
                 <geometry>
-                    <cylinder radius="0.1" length="0.05"/>
+                    <cylinder radius="0.08" length="0.05"/>
                 </geometry>
             </visual>
@@ -12,5 +12,5 @@
                 <origin xyz="0.0 0.0 0.0" rpy="0.0 1.507 1.507"/>
                 <geometry>
-                    <cylinder radius="0.1" length="0.05"/>
+                    <cylinder radius="0.08" length="0.05"/>
                 </geometry>
             </collision>
