Commit message: correcting wheels joints

File: my_robot/urdf/my_robot.xacro (robot description, xacro)
@@ -61,5 +61,5 @@
   <xacro:wheel side="right"/>
   <joint type="continuous" name="left_wheel_hinge">
-            <origin xyz="0 0.19 -0.02" rpy="0 0 0"/>
+            <origin xyz="0 0.175 -0.02" rpy="0 0 0"/>
             <child link="left_wheel"/>
             <parent link="chassis"/>
@@ -69,5 +69,5 @@
           </joint>
   <joint type="continuous" name="right_wheel_hinge">
-            <origin xyz="0 -0.19 -0.02" rpy="0 0 0"/>
+            <origin xyz="0 -0.175 -0.02" rpy="0 0 0"/>
             <child link="right_wheel"/>
             <parent link="chassis"/>
